Commit message: name changed

File: helios_description/urdf/helios_description.xacro (robot description, xacro)
@@ -1,7 +1,7 @@
 <?xml version="1.0" ?>
 <robot name="chipta" xmlns:xacro="http://www.ros.org/wiki/xacro">
-<xacro:include filename="$(find chipta_bot)/urdf/materials.xacro" />
-<xacro:include filename="$(find chipta_bot)/urdf/chipta.ros2control" />
-<xacro:include filename="$(find chipta_bot)/urdf/chipta.gazebo" />
+<xacro:include filename="$(find helios_description)/urdf/materials.xacro" />
+<xacro:include filename="$(find helios_description)/urdf/helios_description.ros2control" />
+<xacro:include filename="$(find helios_description)/urdf/helios_description.gazebo" />
 <link name="base_link">
   <inertial>
@@ -13,5 +13,5 @@
     <origin xyz="0 0 0" rpy="0 0 0"/>
     <geometry>
-      <mesh filename="file://$(find chipta_bot)/meshes/base_link.stl" scale="0.001 0.001 0.001"/>
+      <mesh filename="file://$(find helios_description)/meshes/base_link.stl" scale="0.001 0.001 0.001"/>
     </geometry>
     <material name="purple"/>
@@ -20,5 +20,5 @@
     <origin xyz="0 0 0" rpy="0 0 0"/>
     <geometry>
-      <mesh filename="file://$(find chipta_bot)/meshes/base_link.stl" scale="0.001 0.001 0.001"/>
+      <mesh filename="file://$(find helios_description)/meshes/base_link.stl" scale="0.001 0.001 0.001"/>
     </geometry>
   </collision>
@@ -33,5 +33,5 @@
     <origin xyz="-0.005 -0.0 -0.015" rpy="0 0 0"/>
     <geometry>
-      <mesh filename="file://$(find chipta_bot)/meshes/IMU_v1_1.stl" scale="0.001 0.001 0.001"/>
+      <mesh filename="file://$(find helios_description)/meshes/IMU_v1_1.stl" scale="0.001 0.001 0.001"/>
     </geometry>
     <material name="light_blue"/>
@@ -40,5 +40,5 @@
     <origin xyz="-0.005 -0.0 -0.015" rpy="0 0 0"/>
     <geometry>
-      <mesh filename="file://$(find chipta_bot)/meshes/IMU_v1_1.stl" scale="0.001 0.001 0.001"/>
+      <mesh filename="file://$(find helios_description)/meshes/IMU_v1_1.stl" scale="0.001 0.001 0.001"/>
     </geometry>
   </collision>
@@ -53,5 +53,5 @@
     <origin xyz="0.03 -0.0 -0.018" rpy="0 0 0"/>
     <geometry>
-      <mesh filename="file://$(find chipta_bot)/meshes/GPS_v1_1.stl" scale="0.001 0.001 0.001"/>
+      <mesh filename="file://$(find helios_description)/meshes/GPS_v1_1.stl" scale="0.001 0.001 0.001"/>
     </geometry>
     <material name="green"/>
@@ -60,5 +60,5 @@
     <origin xyz="0.03 -0.0 -0.018" rpy="0 0 0"/>
     <geometry>
-      <mesh filename="file://$(find chipta_bot)/meshes/GPS_v1_1.stl" scale="0.001 0.001 0.001"/>
+      <mesh filename="file://$(find helios_description)/meshes/GPS_v1_1.stl" scale="0.001 0.001 0.001"/>
     </geometry>
   </collision>
@@ -73,5 +73,5 @@
     <origin xyz="-0.1125 0.0015 -0.04" rpy="0 0 0"/>
     <geometry>
-      <mesh filename="file://$(find chipta_bot)/meshes/Lidar_v1_1.stl" scale="0.001 0.001 0.001"/>
+      <mesh filename="file://$(find helios_description)/meshes/Lidar_v1_1.stl" scale="0.001 0.001 0.001"/>
     </geometry>
     <material name="blue"/>
@@ -80,5 +80,5 @@
     <origin xyz="-0.1125 0.0015 -0.04" rpy="0 0 0"/>
     <geometry>
-      <mesh filename="file://$(find chipta_bot)/meshes/Lidar_v1_1.stl" scale="0.001 0.001 0.001"/>
+      <mesh filename="file://$(find helios_description)/meshes/Lidar_v1_1.stl" scale="0.001 0.001 0.001"/>
     </geometry>
   </collision>
@@ -93,5 +93,5 @@
     <origin xyz="-0.064778 -0.085 -0.030131" rpy="0 0 0"/>
     <geometry>
-      <mesh filename="file://$(find chipta_bot)/meshes/Wheel_front_left_1.stl" scale="0.001 0.001 0.001"/>
+      <mesh filename="file://$(find helios_description)/meshes/Wheel_front_left_1.stl" scale="0.001 0.001 0.001"/>
     </geometry>
     <material name="black"/>
@@ -100,5 +100,5 @@
     <origin xyz="-0.064778 -0.085 -0.030131" rpy="0 0 0"/>
     <geometry>
-      <mesh filename="file://$(find chipta_bot)/meshes/Wheel_front_left_1.stl" scale="0.001 0.001 0.001"/>
+      <mesh filename="file://$(find helios_description)/meshes/Wheel_front_left_1.stl" scale="0.001 0.001 0.001"/>
     </geometry>
   </collision>
@@ -113,5 +113,5 @@
     <origin xyz="-0.064778 0.085 -0.030131" rpy="0 0 0"/>
     <geometry>
-      <mesh filename="file://$(find chipta_bot)/meshes/Wheel_front_right_1.stl" scale="0.001 0.001 0.001"/>
+      <mesh filename="file://$(find helios_description)/meshes/Wheel_front_right_1.stl" scale="0.001 0.001 0.001"/>
     </geometry>
     <material name="black"/>
@@ -120,5 +120,5 @@
     <origin xyz="-0.064778 0.085 -0.030131" rpy="0 0 0"/>
     <geometry>
-      <mesh filename="file://$(find chipta_bot)/meshes/Wheel_front_right_1.stl" scale="0.001 0.001 0.001"/>
+      <mesh filename="file://$(find helios_description)/meshes/Wheel_front_right_1.stl" scale="0.001 0.001 0.001"/>
     </geometry>
   </collision>
@@ -133,5 +133,5 @@
     <origin xyz="0.064941 0.085 -0.031781" rpy="0 0 0"/>
     <geometry>
-      <mesh filename="file://$(find chipta_bot)/meshes/Wheel_rear_right_1.stl" scale="0.001 0.001 0.001"/>
+      <mesh filename="file://$(find helios_description)/meshes/Wheel_rear_right_1.stl" scale="0.001 0.001 0.001"/>
     </geometry>
     <material name="black"/>
@@ -140,5 +140,5 @@
     <origin xyz="0.064941 0.085 -0.031781" rpy="0 0 0"/>
     <geometry>
-      <mesh filename="file://$(find chipta_bot)/meshes/Wheel_rear_right_1.stl" scale="0.001 0.001 0.001"/>
+      <mesh filename="file://$(find helios_description)/meshes/Wheel_rear_right_1.stl" scale="0.001 0.001 0.001"/>
     </geometry>
   </collision>
@@ -153,5 +153,5 @@
     <origin xyz="0.064941 -0.085 -0.030131" rpy="0 0 0"/>
     <geometry>
-      <mesh filename="file://$(find chipta_bot)/meshes/Wheel_rear_left_1.stl" scale="0.001 0.001 0.001"/>
+      <mesh filename="file://$(find helios_description)/meshes/Wheel_rear_left_1.stl" scale="0.001 0.001 0.001"/>
     </geometry>
     <material name="black"/>
@@ -160,5 +160,5 @@
     <origin xyz="0.064941 -0.085 -0.030131" rpy="0 0 0"/>
     <geometry>
-      <mesh filename="file://$(find chipta_bot)/meshes/Wheel_rear_left_1.stl" scale="0.001 0.001 0.001"/>
+      <mesh filename="file://$(find helios_description)/meshes/Wheel_rear_left_1.stl" scale="0.001 0.001 0.001"/>
     </geometry>
   </collision>

File: helios_description/urdf/materials.xacro (robot description, xacro)
@@ -1,4 +1,4 @@
 <?xml version="1.0" ?>
-<robot name="chipta" xmlns:xacro="http://www.ros.org/wiki/xacro" >
+<robot name="helios_description" xmlns:xacro="http://www.ros.org/wiki/xacro" >
 <material name="silver">
   <color rgba="0.700 0.700 0.700 1.000"/>

Commit message: mecanum_drive_controller

File: helios_description/urdf/helios_description.xacro (robot description, xacro)
@@ -1,7 +1,20 @@
 <?xml version="1.0" ?>
 <robot name="chipta" xmlns:xacro="http://www.ros.org/wiki/xacro">
+  <xacro:arg name="robot_name" default="helios"/>
+  <xacro:arg name="prefix" default=""/>
+  <xacro:arg name="use_gazebo" default="false"/>
 <xacro:include filename="$(find helios_description)/urdf/materials.xacro" />
-<xacro:include filename="$(find helios_description)/urdf/helios_description.ros2control.xacro" />
+<!-- <xacro:include filename="$(find helios_description)/urdf/helios_description.ros2control.xacro" /> -->
 <xacro:include filename="$(find helios_description)/urdf/helios_description.gazebo" />
+<xacro:include filename="$(find helios_description)/urdf/velocity_control_plugin.urdf.xacro" />
+<xacro:load_velocity_control_plugin use_gazebo="$(arg use_gazebo)"/>
+<xacro:include filename="$(find helios_description)/urdf/gazebo_sim_ros2_control.urdf.xacro" />
+<xacro:load_gazebo_sim_ros2_control_plugin
+  robot_name="$(arg robot_name)"
+  use_gazebo="$(arg use_gazebo)"/>
+<xacro:include filename="$(find helios_description)/urdf/helios_ros2_control.urdf.xacro" />
+<xacro:helios_ros2_control
+  prefix="$(arg prefix)"
+  use_gazebo="$(arg use_gazebo)"/>
 <link name="base_footprint"/>
 <link name="base_link">
@@ -9,12 +22,10 @@
     <origin xyz="0.006285285436363787 2.3801220083224483e-05 0.02118626436883177" rpy="0 0 0"/>
     <mass value="3.955246639227324"/>
-    <inertia ixx="0.017496" iyy="0.029781" izz="0.046394"
-             ixy="2.8e-05" iyz="-1e-06" ixz="3.5e-05"/>
-  </inertial>
-  <visual>
-    <origin xyz="0 0 0" rpy="0 0 0"/>
-    <geometry>
-      <mesh filename="file://$(find helios_description)/meshes/base_link.stl"
-            scale="0.001 0.001 0.001"/>
+    <inertia ixx="0.017496" iyy="0.029781" izz="0.046394" ixy="2.8e-05" iyz="-1e-06" ixz="3.5e-05"/>
+  </inertial>
+  <visual>
+    <origin xyz="0 0 0" rpy="0 0 0"/>
+    <geometry>
+      <mesh filename="file://$(find helios_description)/meshes/base_link.stl" scale="0.001 0.001 0.001"/>
     </geometry>
     <material name="purple"/>
@@ -23,6 +34,5 @@
     <origin xyz="0 0 0" rpy="0 0 0"/>
     <geometry>
-      <mesh filename="file://$(find helios_description)/meshes/base_link.stl"
-            scale="0.001 0.001 0.001"/>
+      <mesh filename="file://$(find helios_description)/meshes/base_link.stl" scale="0.001 0.001 0.001"/>
     </geometry>
   </collision>
@@ -37,6 +47,5 @@
     <origin xyz="-0.005 -0.0 -0.015" rpy="0 0 0"/>
     <geometry>
-      <mesh filename="file://$(find helios_description)/meshes/IMU_v1_1.stl"
-            scale="0.001 0.001 0.001"/>
+      <mesh filename="file://$(find helios_description)/meshes/IMU_v1_1.stl" scale="0.001 0.001 0.001"/>
     </geometry>
     <material name="light_blue"/>
@@ -45,6 +54,5 @@
     <origin xyz="-0.005 -0.0 -0.015" rpy="0 0 0"/>
     <geometry>
-      <mesh filename="file://$(find helios_description)/meshes/IMU_v1_1.stl"
-            scale="0.001 0.001 0.001"/>
+      <mesh filename="file://$(find helios_description)/meshes/IMU_v1_1.stl" scale="0.001 0.001 0.001"/>
     </geometry>
   </collision>
@@ -59,6 +67,5 @@
     <origin xyz="0.03 -0.0 -0.018" rpy="0 0 0"/>
     <geometry>
-      <mesh filename="file://$(find helios_description)/meshes/GPS_v1_1.stl"
-            scale="0.001 0.001 0.001"/>
+      <mesh filename="file://$(find helios_description)/meshes/GPS_v1_1.stl" scale="0.001 0.001 0.001"/>
     </geometry>
     <material name="green"/>
@@ -67,6 +74,5 @@
     <origin xyz="0.03 -0.0 -0.018" rpy="0 0 0"/>
     <geometry>
-      <mesh filename="file://$(find helios_description)/meshes/GPS_v1_1.stl"
-            scale="0.001 0.001 0.001"/>
+      <mesh filename="file://$(find helios_description)/meshes/GPS_v1_1.stl" scale="0.001 0.001 0.001"/>
     </geometry>
   </collision>
@@ -76,12 +82,10 @@
     <origin xyz="-0.0021965658486673423 2.561119446363924e-05 0.007120513681703584" rpy="0 0 0"/>
     <mass value="0.088236472062788"/>
-    <inertia ixx="6e-06" iyy="1.1e-05" izz="1.4e-05"
-             ixy="-0.0" iyz="0.0" ixz="2e-06"/>
+    <inertia ixx="6e-06" iyy="1.1e-05" izz="1.4e-05" ixy="-0.0" iyz="0.0" ixz="2e-06"/>
   </inertial>
   <visual>
     <origin xyz="-0.1125 0.0015 -0.04" rpy="0 0 0"/>
     <geometry>
-      <mesh filename="file://$(find helios_description)/meshes/Lidar_v1_1.stl"
-            scale="0.001 0.001 0.001"/>
+      <mesh filename="file://$(find helios_description)/meshes/Lidar_v1_1.stl" scale="0.001 0.001 0.001"/>
     </geometry>
     <material name="blue"/>
@@ -90,17 +94,9 @@
     <origin xyz="-0.1125 0.0015 -0.04" rpy="0 0 0"/>
     <geometry>
-      <mesh filename="file://$(find helios_description)/meshes/Lidar_v1_1.stl"
-            scale="0.001 0.001 0.001"/>
-    </geometry>
-  </collision>
-</link>
-<!-- ══════════════════════════════════════════════════════════════
-     WHEEL LINKS
-     KEY FIXES:
-       1. collision origin is 0 0 0  (joint handles placement)
-       2. collision geometry is sphere radius=0.04
-       3. inertial origin is 0 0 0
-       4. inertia values correct for sphere m=0.1kg r=0.04m
-     ══════════════════════════════════════════════════════════════ -->
+      <mesh filename="file://$(find helios_description)/meshes/Lidar_v1_1.stl" scale="0.001 0.001 0.001"/>
+    </geometry>
+  </collision>
+</link>
+<!-- ══ FL ══ -->
 <link name="Wheel_front_left_1">
   <inertial>
@@ -118,12 +114,10 @@
     <material name="black"/>
   </visual>
-  <!-- sphere at 0 0 0 — joint origin places it at correct world position -->
-  <collision>
-    <origin xyz="0 0 0" rpy="0 0 0"/>
-    <geometry>
-      <sphere radius="0.04"/>
-    </geometry>
-  </collision>
-</link>
+  <collision>
+    <origin xyz="0 0 0" rpy="0 0 0"/>
+    <geometry><sphere radius="0.04"/></geometry>
+  </collision>
+</link>
+<!-- ══ FR ══ -->
 <link name="Wheel_front_right_1">
   <inertial>
@@ -131,5 +125,5 @@
     <mass value="0.1"/>
     <inertia ixx="6.4e-05" iyy="6.4e-05" izz="6.4e-05"
-             ixy="0.0" iyz="0.0" ixz="-0.0"/>
+             ixy="0.0" iyz="0.0" ixz="0.0"/>
   </inertial>
   <visual>
@@ -143,9 +137,8 @@
   <collision>
     <origin xyz="0 0 0" rpy="0 0 0"/>
-    <geometry>
-      <sphere radius="0.04"/>
-    </geometry>
-  </collision>
-</link>
+    <geometry><sphere radius="0.04"/></geometry>
+  </collision>
+</link>
+<!-- ══ RR ══ -->
 <link name="Wheel_rear_right_1">
   <inertial>
@@ -153,5 +146,5 @@
     <mass value="0.1"/>
     <inertia ixx="6.4e-05" iyy="6.4e-05" izz="6.4e-05"
-             ixy="0.0" iyz="-0.0" ixz="-0.0"/>
+             ixy="0.0" iyz="0.0" ixz="0.0"/>
   </inertial>
   <visual>
@@ -165,9 +158,8 @@
   <collision>
     <origin xyz="0 0 0" rpy="0 0 0"/>
-    <geometry>
-      <sphere radius="0.04"/>
-    </geometry>
-  </collision>
-</link>
+    <geometry><sphere radius="0.04"/></geometry>
+  </collision>
+</link>
+<!-- ══ RL ══ -->
 <link name="Wheel_rear_left_1">
   <inertial>
@@ -175,5 +167,5 @@
     <mass value="0.1"/>
     <inertia ixx="6.4e-05" iyy="6.4e-05" izz="6.4e-05"
-             ixy="0.0" iyz="-0.0" ixz="0.0"/>
+             ixy="0.0" iyz="0.0" ixz="0.0"/>
   </inertial>
   <visual>
@@ -187,36 +179,31 @@
   <collision>
     <origin xyz="0 0 0" rpy="0 0 0"/>
-    <geometry>
-      <sphere radius="0.04"/>
-    </geometry>
-  </collision>
-</link>
-<!-- ══════════════════════════════════════════════════════════════
-     JOINTS — unchanged
-     ══════════════════════════════════════════════════════════════ -->
+    <geometry><sphere radius="0.04"/></geometry>
+  </collision>
+</link>
 <joint name="fixed_base_joint" type="fixed">
-  <parent link="base_footprint"/>
-  <child  link="base_link"/>
-  <origin xyz="0 0 0" rpy="0 0 0"/>
+  <parent link="base_footprint" />
+  <child link="base_link" />
+  <origin xyz="0 0 0" rpy="0 0 0" />
 </joint>
 <joint name="Rigid 14" type="fixed">
   <origin xyz="0.005 0.0 0.015" rpy="0 0 0"/>
   <parent link="base_link"/>
-  <child  link="IMU_v1_1"/>
+  <child link="IMU_v1_1"/>
 </joint>
 <joint name="Rigid 22" type="fixed">
   <origin xyz="-0.03 0.0 0.018" rpy="0 0 0"/>
   <parent link="base_link"/>
-  <child  link="GPS_v1_1"/>
+  <child link="GPS_v1_1"/>
 </joint>
 <joint name="Rigid 23" type="fixed">
   <origin xyz="0.1125 -0.0015 0.04" rpy="0 0 0"/>
   <parent link="base_link"/>
-  <child  link="Lidar_v1_1"/>
+  <child link="Lidar_v1_1"/>
 </joint>
 <joint name="wheel_front_left_joint" type="continuous">
   <origin xyz="0.064778 0.085 0.030131" rpy="0 0 0"/>
   <parent link="base_link"/>
-  <child  link="Wheel_front_left_1"/>
+  <child link="Wheel_front_left_1"/>
   <axis xyz="0.0 1.0 0.0"/>
 </joint>
@@ -224,5 +211,5 @@
   <origin xyz="0.064778 -0.085 0.030131" rpy="0 0 0"/>
   <parent link="base_link"/>
-  <child  link="Wheel_front_right_1"/>
+  <child link="Wheel_front_right_1"/>
   <axis xyz="0.0 1.0 0.0"/>
 </joint>
@@ -230,5 +217,5 @@
   <origin xyz="-0.064941 -0.085 0.031781" rpy="0 0 0"/>
   <parent link="base_link"/>
-  <child  link="Wheel_rear_right_1"/>
+  <child link="Wheel_rear_right_1"/>
   <axis xyz="0.0 1.0 0.0"/>
 </joint>
@@ -236,5 +223,5 @@
   <origin xyz="-0.064941 0.085 0.030131" rpy="0 0 0"/>
   <parent link="base_link"/>
-  <child  link="Wheel_rear_left_1"/>
+  <child link="Wheel_rear_left_1"/>
   <axis xyz="0.0 1.0 0.0"/>
 </joint>

Commit message: push push

File: helios_description/urdf/helios_description.xacro (robot description, xacro)
@@ -7,8 +7,8 @@
 <xacro:include filename="$(find helios_description)/urdf/helios_description.gazebo" />
 <!-- ros2_control hardware interface block -->
-<xacro:include filename="$(find helios_description)/urdf/gazebo_sim_ros2_control.urdf.xacro" />
+<!-- <xacro:include filename="$(find helios_description)/urdf/gazebo_sim_ros2_control.urdf.xacro" /> -->
 <!-- Gazebo plugin that loads gz_ros2_control -->
 <xacro:include filename="$(find helios_description)/urdf/helios_description.ros2control.xacro" />
-<xacro:load_gazebo_sim_ros2_control_plugin robot_name="helios" use_gazebo="true"/>
+<!-- <xacro:load_gazebo_sim_ros2_control_plugin robot_name="helios" use_gazebo="true"/> -->
 <link name="base_footprint"/>
 <link name="base_link">
@@ -143,5 +143,5 @@
   </inertial>
   <visual>
-    <origin xyz="0.064941 0.085 -0.031781" rpy="0 0 0"/>
+    <origin xyz="0.064941 0.085 -0.030131" rpy="0 0 0"/>
     <geometry>
       <mesh filename="file://$(find helios_description)/meshes/Wheel_rear_right_1.stl"
